Commit message: week04: 팀장 10/14 규칙(REP 103·공칭값·영점) 반영 v0 재생성, 골격 대조, 보고서·로그 갱신
- build_v0_urdf.py: cad_frame 고정 변환 1개, 축 직교·좌우 대칭 공칭값, 영점 팔 내림·팔꿈치 전방 굽힘
- verify_robot_v0.py: CAD 자세(yaw +pi/2) 편차표 joint_origin_check.csv, 접촉 0, 2 s 유지 최대 0.056 deg
- check_skeleton_vs_cad.py: 공칭 v0 vs 박종진 골격 8축 축·부호 일치, 앵커 차 <= 1.73 mm
- 노트북 뷰어 캡처 2장 갱신(새 영점), 렌더 4장
- logs/week04.md, notes/09 §10, 4주차 보고서 갱신

Co-Authored-By: Claude Opus 5.5 <noreply@anthropic.com>
Claude-Session: https://claude.ai/code/session_01EMXRjTpmBaPLRBRAVHKhW2

File: sim/robot/our_robot_v0.urdf (robot description, URDF)
Before this commit: robot our_robot_v0, 11 links, 10 joints
Links:
- added link cad_frame
Joints:
- added joint cad_frame_joint: type fixed, parent torso_link, child cad_frame, origin xyz=0 0.11814 0 rpy=1.5708 0 1.5708
- joint left_elbow_joint: axis 0.9997 0 -0.0239 -> 1 0 0; origin xyz=0.01775 0.0001 -0.11546 rpy=0 0 0 -> xyz=0.01775 0 -0.11546 rpy=0 0 0
- joint left_shoulder_roll_joint: axis 1 0 0.0002 -> 1 0 0
- joint left_shoulder_yaw_joint: axis 0.0239 -0.0009 0.9997 -> 0 0 1; origin xyz=-0.02066 1e-05 -0.16015 rpy=0 0 0 -> xyz=-0.02066 0 -0.16015 rpy=0 0 -1.5708
- joint right_elbow_joint: axis 0.9997 0 -0.0239 -> -1 0 0; origin xyz=0.01775 8e-05 -0.11546 rpy=0 0 0 -> xyz=0.01775 0 -0.11546 rpy=0 0 0
- joint right_shoulder_roll_joint: axis 1 0 0.0002 -> -1 0 0
- joint right_shoulder_yaw_joint: axis 0.0239 -0.0006 0.9997 -> 0 0 -1; origin xyz=-0.02064 0.00712 -0.15966 rpy=0 0 0 -> xyz=-0.02066 0 -0.16015 rpy=0 0 1.5708
